File: pcb/atari-2600-composite-video-mod.kicad_sch (KiCad schematic)
At the start: 15 parts, among them J1 RF MOD HEADER, J2 OUTPUT, J3 AUDIO IN, Q1 2N3904, Q2 2N3906

Commit message: Writing comments
Other:
- note added: "Design based on: https://forums.atariage.com/topic/271678-simple-diy-composite-video-mod/"
- note added: "Installation guide: https://forums.atariage.com/topic/301224-composite-mod-for-the-atari-2600-jr-pal-rev-f/"
- title: (none) -> Atari 2600 Composite Video Mod
Changed lines of the file:
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@@
 	(generator_version "8.0")
 	(paper "A5")
+	(title_block
+		(title "Atari 2600 Composite Video Mod")
+		(date "2025-02-06")
+		(rev "0")
+	)
 	(junction
 		(at 53.34 48.26)
@@
 			(width 0)
 			(type default)
+		)
+	)
+	(text "Design based on: https://forums.atariage.com/topic/271678-simple-diy-composite-video-mod/"
+		(exclude_from_sim no)
+		(at 61.976 14.732 0)
+		(effects
+			(font
+				(size 1.27 1.27)
+			)
 		)
 	)
@@
 		(effects
 			(font
+				(size 1.27 1.27)
+			)
+		)
+	)
+	(text "Installation guide: https://forums.atariage.com/topic/301224-composite-mod-for-the-atari-2600-jr-pal-rev-f/"
+		(exclude_from_sim no)
+		(at 70.866 18.034 0)
+		(effects
+			(font
